Commit message: DSR ROS 2 Service Client Test Package operated by unittest

File: dsr_description2/xacro/robotiq_2f.urdf.xacro (robot description, xacro)
@@ -24,5 +24,5 @@
   <joint name="robotiq_coupler_joint" type="fixed">
     <origin xyz="0 0 0.004" rpy="0 0 ${-pi/2.0}" />
-    <parent link="link6"/>
+    <parent link="link_6"/>
     <child link="robotiq_coupler"/>
   </joint>

File: dsr_description2/xacro/robotiq_85_gripper.urdf.xacro (robot description, xacro)
@@ -1,5 +1,5 @@
 <?xml version="1.0"?>
 <robot name="robotiq_85_gripper" xmlns:xacro="http://www.ros.org/wiki/xacro">
-  <xacro:include filename="$(find dsr_description)/xacro/robotiq_85_gripper.transmission.xacro" />
+  <xacro:include filename="$(find dsr_description2)/xacro/robotiq_85_gripper.transmission.xacro" />
   <xacro:macro name="robotiq_85_gripper" params="prefix parent *origin">
     <joint name="${prefix}robotiq_85_base_joint" type="fixed">
@@ -11,10 +11,10 @@
       <visual>
         <geometry>
-          <mesh filename="package://dsr_description/meshes/gripper/robotiq/85_2f/visual/robotiq_85_base_link.dae"/>
-        </geometry>
-      </visual>
-      <collision>
-        <geometry>
-          <mesh filename="package://dsr_description/meshes/gripper/robotiq/85_2f/collision/robotiq_85_base_link.stl"/>
+          <mesh filename="package://dsr_description2/meshes/gripper/robotiq/85_2f/visual/robotiq_85_base_link.dae"/>
+        </geometry>
+      </visual>
+      <collision>
+        <geometry>
+          <mesh filename="package://dsr_description2/meshes/gripper/robotiq/85_2f/collision/robotiq_85_base_link.stl"/>
         </geometry>
       </collision>
@@ -45,10 +45,10 @@
       <visual>
         <geometry>
-          <mesh filename="package://dsr_description/meshes/gripper/robotiq/85_2f/visual/robotiq_85_knuckle_link.dae"/>
-        </geometry>
-      </visual>
-      <collision>
-        <geometry>
-          <mesh filename="package://dsr_description/meshes/gripper/robotiq/85_2f/collision/robotiq_85_knuckle_link.stl"/>
+          <mesh filename="package://dsr_description2/meshes/gripper/robotiq/85_2f/visual/robotiq_85_knuckle_link.dae"/>
+        </geometry>
+      </visual>
+      <collision>
+        <geometry>
+          <mesh filename="package://dsr_description2/meshes/gripper/robotiq/85_2f/collision/robotiq_85_knuckle_link.stl"/>
         </geometry>
       </collision>
@@ -64,10 +64,10 @@
       <visual>
         <geometry>
-          <mesh filename="package://dsr_description/meshes/gripper/robotiq/85_2f/visual/robotiq_85_knuckle_link.dae"/>
-        </geometry>
-      </visual>
-      <collision>
-        <geometry>
-          <mesh filename="package://dsr_description/meshes/gripper/robotiq/85_2f/collision/robotiq_85_knuckle_link.stl"/>
+          <mesh filename="package://dsr_description2/meshes/gripper/robotiq/85_2f/visual/robotiq_85_knuckle_link.dae"/>
+        </geometry>
+      </visual>
+      <collision>
+        <geometry>
+          <mesh filename="package://dsr_description2/meshes/gripper/robotiq/85_2f/collision/robotiq_85_knuckle_link.stl"/>
         </geometry>
       </collision>
@@ -93,10 +93,10 @@
       <visual>
         <geometry>
-          <mesh filename="package://dsr_description/meshes/gripper/robotiq/85_2f/visual/robotiq_85_finger_link.dae"/>
-        </geometry>
-      </visual>
-      <collision>
-        <geometry>
-          <mesh filename="package://dsr_description/meshes/gripper/robotiq/85_2f/collision/robotiq_85_finger_link.stl"/>
+          <mesh filename="package://dsr_description2/meshes/gripper/robotiq/85_2f/visual/robotiq_85_finger_link.dae"/>
+        </geometry>
+      </visual>
+      <collision>
+        <geometry>
+          <mesh filename="package://dsr_description2/meshes/gripper/robotiq/85_2f/collision/robotiq_85_finger_link.stl"/>
         </geometry>
       </collision>
@@ -112,10 +112,10 @@
       <visual>
         <geometry>
-          <mesh filename="package://dsr_description/meshes/gripper/robotiq/85_2f/visual/robotiq_85_finger_link.dae"/>
-        </geometry>
-      </visual>
-      <collision>
-        <geometry>
-          <mesh filename="package://dsr_description/meshes/gripper/robotiq/85_2f/collision/robotiq_85_finger_link.stl"/>
+          <mesh filename="package://dsr_description2/meshes/gripper/robotiq/85_2f/visual/robotiq_85_finger_link.dae"/>
+        </geometry>
+      </visual>
+      <collision>
+        <geometry>
+          <mesh filename="package://dsr_description2/meshes/gripper/robotiq/85_2f/collision/robotiq_85_finger_link.stl"/>
         </geometry>
       </collision>
@@ -147,10 +147,10 @@
       <visual>
         <geometry>
-          <mesh filename="package://dsr_description/meshes/gripper/robotiq/85_2f/visual/robotiq_85_inner_knuckle_link.dae"/>
-        </geometry>
-      </visual>
-      <collision>
-        <geometry>
-          <mesh filename="package://dsr_description/meshes/gripper/robotiq/85_2f/collision/robotiq_85_inner_knuckle_link.stl"/>
+          <mesh filename="package://dsr_description2/meshes/gripper/robotiq/85_2f/visual/robotiq_85_inner_knuckle_link.dae"/>
+        </geometry>
+      </visual>
+      <collision>
+        <geometry>
+          <mesh filename="package://dsr_description2/meshes/gripper/robotiq/85_2f/collision/robotiq_85_inner_knuckle_link.stl"/>
         </geometry>
       </collision>
@@ -166,10 +166,10 @@
       <visual>
         <geometry>
-          <mesh filename="package://dsr_description/meshes/gripper/robotiq/85_2f/visual/robotiq_85_inner_knuckle_link.dae"/>
-        </geometry>
-      </visual>
-      <collision>
-        <geometry>
-          <mesh filename="package://dsr_description/meshes/gripper/robotiq/85_2f/collision/robotiq_85_inner_knuckle_link.stl"/>
+          <mesh filename="package://dsr_description2/meshes/gripper/robotiq/85_2f/visual/robotiq_85_inner_knuckle_link.dae"/>
+        </geometry>
+      </visual>
+      <collision>
+        <geometry>
+          <mesh filename="package://dsr_description2/meshes/gripper/robotiq/85_2f/collision/robotiq_85_inner_knuckle_link.stl"/>
         </geometry>
       </collision>
@@ -201,5 +201,5 @@
       <visual>
         <geometry>
-          <mesh filename="package://dsr_description/meshes/gripper/robotiq/85_2f/visual/robotiq_85_finger_tip_link.dae"/>
+          <mesh filename="package://dsr_description2/meshes/gripper/robotiq/85_2f/visual/robotiq_85_finger_tip_link.dae"/>
         </geometry>
       </visual>
@@ -207,5 +207,5 @@
       <collision>
         <geometry>
-          <mesh filename="package://dsr_description/meshes/gripper/robotiq/85_2f/collision/robotiq_85_finger_tip_link.stl"/>
+          <mesh filename="package://dsr_description2/meshes/gripper/robotiq/85_2f/collision/robotiq_85_finger_tip_link.stl"/>
         </geometry>
       </collision>
@@ -221,5 +221,5 @@
       <visual>
         <geometry>
-          <mesh filename="package://dsr_description/meshes/gripper/robotiq/85_2f/visual/robotiq_85_finger_tip_link.dae"/>
+          <mesh filename="package://dsr_description2/meshes/gripper/robotiq/85_2f/visual/robotiq_85_finger_tip_link.dae"/>
         </geometry>
       </visual>
@@ -227,5 +227,5 @@
       <collision>
         <geometry>
-          <mesh filename="package://dsr_description/meshes/gripper/robotiq/85_2f/collision/robotiq_85_finger_tip_link.stl"/>
+          <mesh filename="package://dsr_description2/meshes/gripper/robotiq/85_2f/collision/robotiq_85_finger_tip_link.stl"/>
         </geometry>
       </collision>
